File: memdump_hw.kicad_pcb (KiCad board)
At the start: 2 copper layers, 56.1 x 86.1 mm, 76 parts, among them J1 USB_C_USB2.0, J2 SWD, J3 LEVEL, J4 BOOT0, Q1 SI4800, SW1 RESET, U1 AMS1117-3.3, U2 STM32F103C8, U3 74HC595, U4 74HC595, U5 74HC595, U6 DIP28/32, Y1 12M

Commit message: fix: USB-C to UFP
Parts:
- added D4: LED, LED_SMD:LED_0805_2012Metric_Pad1.15x1.40mm_HandSolder, F.Cu at (197.6, 62.5)
- added G***: LOGO, LOGO, B.Cu at (177.8, 102.6)
- added G***: LOGO, LOGO, B.Cu at (196.7, 81.0)
- added G***: LOGO, LOGO, B.Cu at (176.8, 64.8)
- added R12: 470, Resistor_SMD:R_0805_2012Metric_Pad1.20x1.40mm_HandSolder, F.Cu at (200.4, 62.5)
- moved R30 2.54 mm to (206.2, 92.5)
- moved R5 2.05 mm to (216.4, 114.0)
- moved U4 0.25 mm to (200.7, 100.1)
- turned R3 to 180 degrees
- renumbered C11 to C10, C12 to C11, C13 to C12, C14 to C13, C15 to C14, C16 to C15, C18 to C16, C3 to C2, C4 to C3, C5 to C4, C6 to C5, C7 to C6, C8 to C7, C2 to C8, C10 to C9, J4 to J3, J3 to J4, R40 to R10, R42 to R11, R30 to R13, R31 to R14, R32 to R15, R8 to R16, R9 to R17, R10 to R18, R11 to R19, R12 to R20, R13 to R21, R14 to R22, R15 to R23, R16 to R24, R17 to R25, R18 to R26, R19 to R27, R20 to R28, R21 to R29, R25 to R30, R23 to R31, R24 to R32, R26 to R33, R27 to R34, R28 to R35, R29 to R36, R33 to R37, R34 to R38, R35 to R39, R36 to R40, R37 to R41, R38 to R42, R39 to R43, R22 to R8, R41 to R9
Connections:
- net A13+NWE renamed A13
- D3 pad 1: A14+VCC_28 -> A17+VCC_28
- J1 pad A5: Net-(J1-PadA5) -> Net-(R3-Pad1)
- J1 pad B5: Net-(J1-PadA5) -> Net-(R3-Pad1)
- Q1 pad 5: A14+VCC_28 -> A17+VCC_28
- Q1 pad 6: A14+VCC_28 -> A17+VCC_28
- Q1 pad 7: A14+VCC_28 -> A17+VCC_28
- Q1 pad 8: A14+VCC_28 -> A17+VCC_28
- R3 pad 1: +5V -> Net-(R3-Pad1)
- R3 pad 2: Net-(J1-PadA5) -> GND
- R30 pad 1: A17 -> A14
- R30 pad 2: Net-(R25-Pad2) (its old number) -> Net-(R30-Pad2)
- R8 pad 1: A14 -> A17
- U4 pad 15: A14 -> A17
- U4 pad 2: A17 -> A14
- U6 pad 29: A14+VCC_28 -> Net-(R30-Pad2)
- U6 pad 30: Net-(R25-Pad2) (its old number) -> A17+VCC_28
Routing:
- net A14+VCC_28: track 16.1 -> 0.00 mm
- net A17+VCC_28: track 0.00 -> 15.0 mm
- net Net-(R3-Pad1): track 0.00 -> 9.84 mm
- net Net-(J1-PadA5): track 9.84 -> 0.00 mm
- net ACT: track 0.00 -> 5.82 mm
- net +5V: track 49.0 -> 43.3 mm
- net A17: track 8.30 -> 5.09 mm, vias 1 -> 0
- net Net-(D4-Pad2): track 0.00 -> 2.80 mm
- net Net-(R30-Pad2): track 0.00 -> 2.56 mm
- net Net-(R25-Pad2) (its old number): track 2.56 -> 0.00 mm
- net Net-(J3-Pad2): track 5.18 -> 4.08 mm
- net /BOOT0: track 21.3 -> 20.8 mm
- net A14: track 5.09 -> 5.46 mm, vias 0 -> 1
Other:
- board text added: "0"
- board text added: "1"
- board text added: "3V3"
- board text added: "5V"
- board text added: "GND"
- board text added: "SWCLK"
- board text added: "SWDIO"
- board text added: "memdump by HA5PLS"
